File: pcb/M_U_M.kicad_sch (KiCad schematic)
At the start: 28 parts, among them J1 Conn_01x04, SW1 RotaryEncoder_Switch, SW10 SW_Push, SW11 SW_Push, SW12 SW_Push, SW2 RotaryEncoder_Switch, SW3 SW_Push, SW4 SW_Push, SW5 SW_Push, SW6 SW_Push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

Commit message: we updated and routed
Parts:
- RV1, RV2: footprint Potentiometer_THT:Potentiometer_Alps_RK09K_Single_Horizontal -> Potentiometer_THT:Potentiometer_Bourns_PTA6043_Single_Slide
Connections:
- net POT1: now also U1.20 (GP29); no longer U1.19 (GP28)
- net POT2: now also U1.19 (GP28); no longer U1.20 (GP29)
- net R1A: now also U1.12 (GP11); no longer U1.13 (GP12)
- net R1B: now also U1.13 (GP12); no longer U1.14 (GP13)
- net R2A: now also U1.14 (GP13); no longer U1.15 (GP14)
- net R2B: now also U1.15 (GP14); no longer U1.16 (GP15)
- net ROW0: now also U1.7 (GP6); no longer U1.4 (GP3)
- net ROW1: now also U1.6 (GP5); no longer U1.5 (GP4)
- net ROW2: now also U1.5 (GP4); no longer U1.6 (GP5)
- net ROW3: now also U1.4 (GP3); no longer U1.7 (GP6)
- net SCL: now also U1.17 (GP26); no longer U1.8 (GP7)
- net SDA: now also U1.16 (GP15); no longer U1.9 (GP8)
Changed lines of the file:
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@@
 	(wire
 		(pts
+			(xy 262.89 39.37) (xy 269.24 39.37)
+		)
+		(stroke
+			(width 0)
+			(type default)
+		)
+	)
+	(wire
+		(pts
 			(xy 262.89 46.99) (xy 269.24 46.99)
 		)
@@
 	(wire
 		(pts
-			(xy 223.52 57.15) (xy 227.33 57.15)
-		)
-		(stroke
-			(width 0)
-			(type default)
-		)
-	)
-	(wire
-		(pts
 			(xy 222.25 46.99) (xy 227.33 46.99)
 		)
@@
 	(wire
 		(pts
-			(xy 223.52 54.61) (xy 227.33 54.61)
+			(xy 262.89 52.07) (xy 269.24 52.07)
 		)
 		(stroke
@@
 		)
 	)
-	(label "R2B"
-		(at 184.15 154.94 0)
+	(label "ROW3"
+		(at 222.25 44.45 0)
 		(effects
 			(font
@@
 		)
 	)
-	(label "R1B"
-		(at 269.24 44.45 180)
+	(label "R2B"
+		(at 184.15 154.94 0)
 		(effects
 			(font
 				(size 1.27 1.27)
 			)
-			(justify right bottom)
+			(justify left bottom)
 		)
 	)
-	(label "R1S2"
-		(at 231.14 93.98 180)
+	(label "POT2"
+		(at 269.24 57.15 180)
 		(effects
 			(font
@@
 	)
 	(label "R1S2"
-		(at 210.82 138.43 180)
+		(at 231.14 93.98 180)
 		(effects
 			(font
@@
 		)
 	)
-	(label "R2S2"
-		(at 243.84 93.98 180)
+	(label "R1A"
+		(at 269.24 39.37 180)
 		(effects
 			(font
@@
 		)
 	)
-	(label "COL1"
-		(at 222.25 39.37 0)
+	(label "R1S2"
+		(at 210.82 138.43 180)
 		(effects
 			(font
 				(size 1.27 1.27)
 			)
-			(justify left bottom)
+			(justify right bottom)
 		)
 	)
-	(label "ROW1"
-		(at 222.25 46.99 0)
+	(label "R2S2"
+		(at 243.84 93.98 180)
 		(effects
 			(font
 				(size 1.27 1.27)
 			)
-			(justify left bottom)
+			(justify right bottom)
 		)
 	)
-	(label "R2A"
-		(at 269.24 46.99 180)
+	(label "COL1"
+		(at 222.25 39.37 0)
 		(effects
 			(font
 				(size 1.27 1.27)
 			)
-			(justify right bottom)
+			(justify left bottom)
 		)
 	)
@@
 		)
 	)
-	(label "ROW3"
-		(at 222.25 52.07 0)
-		(effects
-			(font
-				(size 1.27 1.27)
-			)
-			(justify left bottom)
-		)
-	)
 	(label "COL0"
 		(at 222.25 36.83 0)
@@
 		)
 	)
-	(label "POT2"
-		(at 269.24 59.69 180)
+	(label "R2A"
+		(at 269.24 44.45 180)
 		(effects
 			(font
@@
 		)
 	)
-	(label "R1A"
-		(at 269.24 41.91 180)
+	(label "SCL"
+		(at 269.24 52.07 180)
 		(effects
 			(font
@@
 		)
 	)
-	(label "R2A"
-		(at 184.15 149.86 0)
+	(label "SDA"
+		(at 269.24 49.53 180)
 		(effects
 			(font
 				(size 1.27 1.27)
 			)
-			(justify left bottom)
+			(justify right bottom)
 		)
 	)
-	(label "R1B"
-		(at 184.15 138.43 0)
+	(label "ROW2"
+		(at 222.25 46.99 0)
 		(effects
 			(font
@@
 		)
 	)
-	(label "R1S1"
-		(at 226.06 95.25 180)
+	(label "R2B"
+		(at 269.24 46.99 180)
 		(effects
 			(font
@@
 		)
 	)
-	(label "R2B"
-		(at 269.24 49.53 180)
+	(label "R2A"
+		(at 184.15 149.86 0)
 		(effects
 			(font
 				(size 1.27 1.27)
 			)
-			(justify right bottom)
+			(justify left bottom)
 		)
 	)
-	(label "R2S1"
-		(at 210.82 149.86 180)
+	(label "POT1"
+		(at 269.24 59.69 180)
 		(effects
 			(font
@@
 		)
 	)
-	(label "POT2"
-		(at 182.88 102.87 180)
+	(label "ROW0"
+		(at 222.25 52.07 0)
 		(effects
 			(font
 				(size 1.27 1.27)
 			)
-			(justify right bottom)
+			(justify left bottom)
 		)
 	)
-	(label "SDA"
-		(at 172.72 142.24 180)
+	(label "R1B"
+		(at 184.15 138.43 0)
+		(effects
+			(font
+				(size 1.27 1.27)
+			)
+			(justify left bottom)
+		)
+	)
+	(label "R1S1"
+		(at 226.06 95.25 180)
 		(effects
 			(font
@@
 		)
 	)
-	(label "ROW3"
-		(at 270.51 157.48 180)
+	(label "R2S1"
+		(at 210.82 149.86 180)
 		(effects
 			(font
@@
 		)
 	)
-	(label "COL2"
-		(at 246.38 78.74 270)
+	(label "POT2"
+		(at 182.88 102.87 180)
 		(effects
 			(font
@@
 		)
 	)
-	(label "POT1"
-		(at 212.09 102.87 180)
+	(label "SDA"
+		(at 172.72 142.24 180)
 		(effects
 			(font
@@
 		)
 	)
-	(label "ROW2"
+	(label "ROW1"
 		(at 222.25 49.53 0)
 		(effects
@@
 		)
 	)
-	(label "R2S1"
-		(at 238.76 95.25 180)
+	(label "ROW3"
+		(at 270.51 157.48 180)
 		(effects
 			(font
@@
 		)
 	)
-	(label "POT1"
-		(at 269.24 57.15 180)
+	(label "R1B"
+		(at 269.24 41.91 180)
 		(effects
 			(font
@@
 		)
 	)
-	(label "SCL"
-		(at 223.52 54.61 0)
+	(label "COL2"
+		(at 246.38 78.74 270)
 		(effects
 			(font
 				(size 1.27 1.27)
 			)
-			(justify left bottom)
+			(justify right bottom)
 		)
 	)
-	(label "SDA"
-		(at 223.52 57.15 0)
+	(label "POT1"
+		(at 212.09 102.87 180)
 		(effects
 			(font
 				(size 1.27 1.27)
 			)
-			(justify left bottom)
+			(justify right bottom)
 		)
 	)
-	(label "R1S1"
-		(at 210.82 133.35 180)
+	(label "R2S1"
+		(at 238.76 95.25 180)
 		(effects
 			(font
@@
 		)
 	)
-	(label "ROW0"
-		(at 222.25 44.45 0)
+	(label "R1S1"
+		(at 210.82 133.35 180)
 		(effects
 			(font
 				(size 1.27 1.27)
 			)
-			(justify left bottom)
+			(justify right bottom)
 		)
 	)
@@
 			)
 		)
-		(property "Footprint" "Potentiometer_THT:Potentiometer_Alps_RK09K_Single_Horizontal"
+		(property "Footprint" "Potentiometer_THT:Potentiometer_Bourns_PTA6043_Single_Slide"
 			(at 172.72 102.87 0)
 			(effects
@@
 			)
 		)
-		(property "Footprint" "Potentiometer_THT:Potentiometer_Alps_RK09K_Single_Horizontal"
+		(property "Footprint" "Potentiometer_THT:Potentiometer_Bourns_PTA6043_Single_Slide"
 			(at 201.93 102.87 0)
 			(effects
